File: Hardware/Basic/Top/BuddyBand-BASIC-TOP.brd (EAGLE design)
At the start: 38 x 38 mm, 51 parts, among them SW1 SWITCH.MOM, SW6 SWITCH.MOM, U2 NRF52832_MODULE_MDBT42, U4 PCF8523

Commit message: In process of working on Take 003 video.
Parts:
- removed LDO2: MIC5504, LinnesLab-Power:SOT23-5
- removed SW6: SWITCH.MOM, LinnesLab-Switches:TACTILE_SWITCH_SMD_6.2MM_TALL
- added C22: 100n, LinnesLab-Passives:C0603
- added C23, C24: 47p, LinnesLab-Passives:C0603
- added J1: (no value), LinnesLab-Connectors:1X07_1.27MM
- added JP2: (no value), LinnesLab-Switches:SMT-JUMPER_2_NO_SILK
- added LDO1: MIC5504, LinnesLab-Power:SOT23-5
- added LED5: RED, LinnesLab-LED:LED-0603
- added LED6: YELLOW, LinnesLab-LED:LED-0603
- added R1, R2: 0, LinnesLab-Passives:R0603
- added R17, R18: 27, LinnesLab-Passives:R0603
- added R19, R20: 1k, LinnesLab-Passives:R0603
- added SW2: SWITCH.MOM, LinnesLab-Switches:TACTILE_SWITCH_SMD_6.2MM_TALL
- added U5: FT231XS, LinnesLab-DigitalIC:SSOP20_L
- R8, R9: value 10k -> 10K
- moved XTAL3 45.9 mm to (35.2, -5.13)
- moved U4 45.6 mm to (39.5, -6.38)
- moved R9 39.5 mm to (-5.03, -11.2), turned to 0 degrees
- moved R8 37.1 mm to (-5.03, -8.51), turned to 0 degrees
- moved R13 24.4 mm to (15.9, -11.4)
- moved CHRG2 19.8 mm to (28.5, -5.99)
- moved C21 19.7 mm to (12.6, -10.9)
- moved D5 19.7 mm to (23.1, -8.15)
- moved D4 18.4 mm to (22.1, -5.59)
- moved R14 17.8 mm to (9.04, -6.65)
- moved R12 16.4 mm to (9.22, -11.0)
- moved C20 14.5 mm to (11.5, -3.25)
- moved C5 13.9 mm to (13.5, -2.67)
- moved R15 13.9 mm to (17.6, -2.46)
- moved C6 13.4 mm to (15.6, -1.98)
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Connections:
- net DC.OLED renamed D4/DC.OLED
- removed net BATT: R13.1, R14.2
- removed net CD1: SD2.CD1
- removed net CHRG.STAT: CHRG2.1, R12.1
- removed net CS.OLED: U3.13
- removed net RESET.OLED: U3.14
- removed net RXD: U2.21
- removed net SD.CS: SD2.2
- removed net SW1: SW1.A1, SW6.A1
- removed net TXD: U2.19
- new net !CTS: JP2.2, U5.9
- new net A4/BATT: R13.1, R14.2, U2.5
- new net A6/TIA: J1.6, U2.7
- new net A7/PPG: J1.7, U2.8
- new net D11/SW1: SW1.A1, U2.25
- new net D15/SW2: SW2.A1, U2.29
- new net D16/CS.OLED: U2.30, U3.13
- new net D27/CHRG.STATUS: CHRG2.1, R12.1, U2.4
- new net D29/LED.CTRL: J1.5, U2.6
- new net D3/RESET.OLED: U2.16, U3.14
- new net D5/CD1: SD2.CD1, U2.18
- new net D7/SD.CS: SD2.2, U2.20
- new net FT3V3: U5.13
- new net N$16: U2.17
- new net N$23: R17.2, U5.12
- new net N$24: R18.2, U5.11
- new net N$25: LED5.C, R19.2
- new net N$26: LED6.C, R20.2
- new net RXD.FT: R2.1, U5.4
- new net RXD.NFR: R1.2, U2.21
- new net RXLED: R19.1, U5.17
- new net TXD.FT: R1.1, U5.20
- new net TXD.NFR: R2.2, U2.19
- new net TXLED: R20.1, U5.10
- net 3.3V: now also C22.2, J1.4, LDO1.5, LED5.A, LED6.A, U5.14, U5.3; no longer LDO2.5
- net DTR: now also U5.1
- net GND: now also C22.1, C23.2, C24.1, J1.3, JP2.1, LDO1.2, SW2.B1, SW2.B2, U5.16, U5.6; no longer LDO2.2, SW6.B1, SW6.B2
- net SCL: now also J1.2, R9.1; no longer R8.1
- net SDA: now also J1.1, R8.1; no longer R9.1
- net USB+: now also C23.1, R18.1
- net USB-: now also C24.2, R17.1
- net VIN: now also LDO1.1, LDO1.3; no longer LDO2.1, LDO2.3
- net V_USB: now also U5.15

Commit message: Finished take 5 working on take 6
Parts:
- removed C10, C11: 300p, LinnesLab-Passives:C0603
- removed C21: 4.7u, LinnesLab-Passives:C0603
- removed C22: 100n, LinnesLab-Passives:C0603
- removed C23, C24: 47p, LinnesLab-Passives:C0603
- removed CHRG2: MCP73831, LinnesLab-Power:SOT23-5
- removed CORTEX1: CORTEX_DEBUG_PTH, LinnesLab-Connectors:2X5-PTH-1.27MM
- removed D4, D5: (no value), LinnesLab-DiscreteSemi:USC
- removed JP2: (no value), LinnesLab-Switches:SMT-JUMPER_2_NO_SILK
- removed L2: 10u, LinnesLab-Passives:L0603
- removed LED5: RED, LinnesLab-LED:LED-0603
- removed LED6: YELLOW, LinnesLab-LED:LED-0603
- removed R19, R20: 1k, LinnesLab-Passives:R0603
- removed R9: 10K, LinnesLab-Passives:R0603
- removed U3: (no value), LinnesLab-Displays:UG-2864HSWEG01_0.96IN_NO-WRAPAROUND
- removed U5: FT231XS, LinnesLab-DigitalIC:SSOP20_L
- removed USB2: USB.MICRO-BIGGERPADS, LinnesLab-Connectors:USB-MICRO-01.BIGGERPADS
- removed XTAL2: 32.768kHz, LinnesLab-Clocks:2-SMD.NOLEAD.2.0MMTO1.2MM
- removed XTAL3: 32.7680kHz, LinnesLab-Clocks:2-SMD.NOLEAD.2.0MMTO1.2MM
- added C1: 47p, LinnesLab-Passives:C0603
- added C3: 1u, LinnesLab-Passives:C0603
- added C4: 100n, LinnesLab-Passives:C0603
- added CHRG1: MCP73831, LinnesLab-Power:SOT23-5
- added D2, D3: (no value), LinnesLab-DiscreteSemi:USC
- added DEBUG1: CORTEX_DEBUG_PTH, LinnesLab-Connectors:2X5-PTH-1.27MM
- added JP1: (no value), LinnesLab-Switches:SMT-JUMPER_2_NO_SILK
- added L1: 10u, LinnesLab-Passives:L0603
- added LED1: RED, LinnesLab-LED:LED-0603
- added LED2: YELLOW, LinnesLab-LED:LED-0603
- added R10: 1k, LinnesLab-Passives:R0603
- added R16: 10k, LinnesLab-Passives:R0603
- added U1: FT231XS, LinnesLab-DigitalIC:SSOP20_L
- added USB1: USB.MICRO-BIGGERPADS, LinnesLab-Connectors:USB-MICRO-01.BIGGERPADS
- added XTAL1: 32.768kHz, LinnesLab-Clocks:2-SMD.NOLEAD.2.0MMTO1.2MM
- C12: value 10u -> 1u; device LinnesLab-Passives:C0805 -> LinnesLab-Passives:C0603
- C13: value 2.2uF -> 4.7u; device LinnesLab-Passives:C0402 -> LinnesLab-Passives:C0603
- C15: value 2.2uF -> 10uF; device LinnesLab-Passives:C0402 -> LinnesLab-Passives:C0603
- C16: value 10uF -> 2.2uF; device LinnesLab-Passives:C0603 -> LinnesLab-Passives:C0402
- C2: value 1u -> 47p
- C20: value 4.7u -> 2.2uF; device LinnesLab-Passives:C0603 -> LinnesLab-Passives:C0402
- C5: value 1u -> 10u; device LinnesLab-Passives:C0603 -> LinnesLab-Passives:C0805
- C6: value 1u -> (none)
- C7: value 1u -> 4.7u
- C8: value (none) -> 1u
- R1, R2: value 0 -> 10K
- R11: value (none) -> 100k
- R13, R14: value 100k -> 0
- R15: value 100k -> 1k
- R17: value 27 -> 10k
- R18: value 27 -> 390k
- R3, R4: value 1k -> 27
- R5: value 10k -> 100k
- R6: value 10k -> 1k
- R7: value 390k -> 1k
- R8: value 10K -> (none)
- SW1, SW2: value SWITCH.MOM -> (none); device LinnesLab-Switches:TACTILE_SWITCH_SMD_6.2MM_TALL -> LinnesLab-Switches:BUTTON-GULLWING
- SW3, SW4: value (none) -> SWITCH.MOM; device LinnesLab-Switches:BUTTON-GULLWING -> LinnesLab-Switches:TACTILE_SWITCH_SMD_6.2MM_TALL
- U4: value PCF8523 -> (none); device LinnesLab-Clocks:SO8 -> LinnesLab-Displays:UG-2864HSWEG01_0.96IN_NO-WRAPAROUND
- moved R17 47.2 mm to (15.4, 22.0), turned to 270 degrees
- moved D1 42.3 mm to (8.29, 3.28), flipped to the bottom, turned to 270 degrees
- moved R1 42.0 mm to (3.84, 39.4)
- moved R2 42.0 mm to (3.84, 36.7)
- moved R4 37.8 mm to (10.9, 3.01)
- moved R5 35.3 mm to (11.6, 8.04), flipped to the bottom, turned to 270 degrees
- moved R3 35.0 mm to (10.9, 4.89)
- moved U4 34.0 mm to (18.5, 20.4)
- moved R15 32.8 mm to (35.6, 24.9)
- moved R18 31.7 mm to (31.9, 19.0), turned to 270 degrees
- moved R12 31.6 mm to (2.02, 19.8), turned to 90 degrees
- moved SW1 31.0 mm to (35.0, 35.7)
- moved SW3 30.8 mm to (31.7, 4.85), turned to 180 degrees
- moved C5 30.2 mm to (16.7, 27.4), turned to 0 degrees
- moved C2 26.3 mm to (13.5, 2.58), turned to 270 degrees
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- renumbered SD2 to SD1
Connections:
- removed net N$19: U4.2, XTAL3.P$1
- removed net N$20: U4.1, XTAL3.P$2
- removed net VBAT: U4.3
- net !CTS: now also JP1.2, U1.9; no longer JP2.2, U5.9
- net 3.3V: now also C12.1, C20.2, C4.2, C5.2, D3.-, DEBUG1.1, LED1.A, LED2.A, R1.2, R16.2, R2.2, U1.14, U1.3, U4.6, U4.9; no longer C12.2, C17.2, C2.1, C22.2, C6.1, CORTEX1.1, D1.-, LED5.A, LED6.A, R15.2, R5.2, R8.2, R9.2, U3.6, U3.9, U4.8, U5.14, U5.3
- net A4/BATT: now also R11.1, R12.2; no longer R13.1, R14.2
- net D11/SW1: now also SW3.A1; no longer SW1.A1
- net D15/SW2: now also SW4.A1; no longer SW2.A1
- net D16/CS.OLED: now also U4.13; no longer U3.13
- net D27/CHRG.STATUS: now also CHRG1.1, R5.1; no longer CHRG2.1, R12.1
- net D3/RESET.OLED: now also U4.14; no longer U3.14
- net D4/DC.OLED: now also U4.15; no longer U3.15
- net DFU: now also SW1.3; no longer SW3.3
- net DTR: now also U1.1; no longer U5.1
- net FT3V3: now also U1.13; no longer U5.13
- net GND: now also C1.1, C12.2, C13.2, C15.1, C20.1, C3.2, C4.1, C6.1, C7.1, CHRG1.2, DEBUG1.3, DEBUG1.5, DEBUG1.7, DEBUG1.9, JP1.1, R12.1, R17.1, R18.2, R8.1, SW1.1, SW2.3, SW3.B1, SW4.B1, U1.16, U1.6, U4.1, U4.10, U4.12, U4.29, U4.30, U4.8, USB1.5, USB1.S1, USB1.S2, USB1.S3, USB1.S4, USB1.S5, USB1.S6; no longer C10.2, C11.2, C12.1, C16.1, C18.1, C20.2, C21.1, C22.1, C23.2, C24.1, C6.2, C7.2, CHRG2.2, CORTEX1.3, CORTEX1.5, CORTEX1.7, CORTEX1.9, JP2.1, R11.1, R14.1, R15.1, R6.1, R7.2, SW1.B1, SW1.B2, SW2.B1, SW2.B2, SW3.1, SW4.3, U3.1, U3.10, U3.12, U3.29, U3.30, U3.8, U4.4, U5.16, U5.6, USB2.5, USB2.S1, USB2.S2, USB2.S3, USB2.S4, USB2.S5, USB2.S6
- net LED1: now also R10.2; no longer R3.2
- net LED2: now also R15.2; no longer R4.2
- net MOSI: now also U4.19; no longer U3.19
- net N$1: now also R17.2, U4.11; no longer R6.2, U3.11
- net N$10: now also R15.1; no longer R4.1
- net N$11: now also L1.1; no longer L2.1
- net N$12: now also C3.1, L1.2; no longer C7.1, L2.2
- net N$13: now also C15.2, U4.28; no longer C16.2, U3.28
- net N$14: now also DEBUG1.8; no longer CORTEX1.8
- net N$15: now also C17.2, U4.27; no longer C18.2, U3.27
- net N$17: now also CHRG1.5, R8.2; no longer CHRG2.5, R11.2
- net N$2: now also R18.1, U4.26; no longer R7.1, U3.26
- net N$23: now also R3.2, U1.12; no longer R17.2, U5.12
- net N$24: now also R4.2, U1.11; no longer R18.2, U5.11
- net N$25: now also LED1.C, R6.2; no longer LED5.C, R19.2
- net N$26: now also LED2.C, R7.2; no longer LED6.C, R20.2
- net N$3: now also C18.2, U4.2; no longer C13.2, U3.2
- net N$4: now also C6.2, XTAL1.P$1; no longer C8.2, XTAL2.P$1
- net N$5: now also C18.1, U4.3; no longer C13.1, U3.3
- net N$6: now also XTAL1.P$2; no longer XTAL2.P$2
- net N$7: now also C16.2, U4.4; no longer C15.2, U3.4
- net N$8: now also C16.1, U4.5; no longer C15.1, U3.5
- net N$9: now also R10.1; no longer R3.1
- net P0.09/NFC1: no longer C11.1
- net P0.10/NFC2: no longer C10.1
- net RESET: now also D3.+, DEBUG1.10, R16.1, SW2.1; no longer CORTEX1.10, D1.+, R5.1, SW4.1
- net RXD.FT: now also R14.1, U1.4; no longer R2.1, U5.4
- net RXD.NFR: now also R13.2; no longer R1.2
- net RXLED: now also R6.1, U1.17; no longer R19.1, U5.17
- net SCK: now also U4.18; no longer U3.18
- net SCL: now also R2.1; no longer R9.1, U4.6
- net SDA: now also R1.1; no longer R8.1, U4.5
- net SWCLK: now also DEBUG1.4; no longer CORTEX1.4
- net SWDIO: now also DEBUG1.2; no longer CORTEX1.2
- net SWO: now also DEBUG1.6; no longer CORTEX1.6
- net TXD.FT: now also R13.1, U1.20; no longer R1.1, U5.20
- net TXD.NFR: now also R14.2; no longer R2.2
- net TXLED: now also R7.1, U1.10; no longer R20.1, U5.10
- net USB+: now also C2.1, R4.1, USB1.3; no longer C23.1, R18.1, USB2.3
- net USB-: now also C1.2, R3.1, USB1.2; no longer C24.2, R17.1, USB2.2
- net VIN: now also C7.2, C8.2, CHRG1.4, D1.-, D2.-, R5.2; no longer C21.2, C5.2, CHRG2.4, D4.-, D5.-, R12.2
- net VLIPO: now also C13.1, CHRG1.3, D1.+, R11.2; no longer C20.1, CHRG2.3, D4.+, R13.2
- net V_USB: now also D2.+, U1.15, USB1.1; no longer D5.+, U5.15, USB2.1
Routing:
- net GND: track 0.00 -> 33.1 mm, vias 0 -> 18
- net VLIPO: track 0.00 -> 22.4 mm
- net USB-: track 0.00 -> 17.5 mm, vias 0 -> 1
- net VIN: track 0.00 -> 14.2 mm
- net USB+: track 0.00 -> 13.8 mm, vias 0 -> 1
- net RESET: track 0.00 -> 12.0 mm
- net SWO: track 0.00 -> 11.2 mm, vias 0 -> 1
- net SWCLK: track 0.00 -> 10.3 mm
- net N$17: track 0.00 -> 9.31 mm
- net N$2: track 0.00 -> 7.90 mm
- net N$4: track 0.00 -> 7.53 mm
- net LED2: track 0.00 -> 7.07 mm
- net N$6: track 0.00 -> 6.78 mm
- net SWDIO: track 0.00 -> 6.48 mm, vias 0 -> 1
- net N$13: track 0.00 -> 4.69 mm
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- added copper zone on layer 1, net 3.3V
- added copper zone on layer 16, net GND

Commit message: doing take 7. have trouble with wiring
Parts:
- removed SD1: (no value), LinnesLab-Connectors:MICROSD
- moved R14 13.6 mm to (18.7, 10.7)
- moved C17 11.5 mm to (30.4, 16.9), turned to 180 degrees
- moved R13 10.2 mm to (18.8, 8.95)
- moved SW4 9.92 mm to (31.7, 4.23)
- moved SW3 9.73 mm to (22.0, 4.25)
- moved R1 6.97 mm to (1.63, 32.8), turned to 270 degrees
- moved R2 3.95 mm to (3.17, 32.8), turned to 270 degrees
- moved C5 3.32 mm to (17.9, 30.5)
- moved C4 2.69 mm to (2.63, 12.0), turned to 180 degrees
- moved JP1 2.27 mm to (1.66, 2.56), turned to 90 degrees
- moved C3 2.26 mm to (18.3, 27.5), turned to 180 degrees
- moved L1 1.72 mm to (18.4, 26.1), turned to 0 degrees
- moved D3 1.19 mm to (35.2, 13.7)
- moved R16 1.15 mm to (35.3, 15.2)
- moved C14 1.12 mm to (35.4, 12.4)
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Connections:
- removed net A6/TIA: J1.6, U2.7
- removed net A7/PPG: J1.7, U2.8
- removed net CD2: SD1.CD2
- removed net D29/LED.CTRL: J1.5, U2.6
- removed net N$16: U2.17
- new net A5/TIA: J1.6, U2.6
- new net A7/BATT: R11.1, R12.2, U2.8
- new net D30/LED.CTRL: J1.5, U2.7
- net 3.3V: no longer SD1.4
- net A4/BATT: now also J1.7; no longer R11.1, R12.2
- net D4/DC.OLED: now also U2.17
- net D5/CD1: no longer SD1.CD1
- net D7/SD.CS: no longer SD1.2
- net GND: no longer SD1.6, SD1.MT1, SD1.MT2
- net MISO: no longer SD1.7
- net MOSI: no longer SD1.3
- net SCK: no longer SD1.5
Routing:
- net 3.3V: track 2.44 -> 48.7 mm, vias 1 -> 6
- net DTR: track 0.00 -> 42.3 mm, vias 0 -> 2
- net GND: track 33.1 -> 63.8 mm, vias 18 -> 22
- net RXD.NFR: track 0.00 -> 24.2 mm, vias 0 -> 2
- net SDA: track 0.00 -> 23.4 mm, vias 0 -> 1
- net D15/SW2: track 0.00 -> 23.2 mm, vias 0 -> 2
- net A7/BATT: track 0.00 -> 22.7 mm, vias 0 -> 2
- net SCL: track 0.00 -> 22.5 mm, vias 0 -> 1
- net D11/SW1: track 0.00 -> 21.5 mm
- net TXD.NFR: track 0.00 -> 19.8 mm, vias 0 -> 2
- net D16/CS.OLED: track 0.00 -> 18.9 mm, vias 0 -> 2
- net SCK: track 0.00 -> 16.3 mm, vias 0 -> 2
- net RXD.FT: track 0.11 -> 16.4 mm
- net RESET: track 12.0 -> 27.0 mm, vias 0 -> 1
- net MOSI: track 0.00 -> 15.0 mm, vias 0 -> 2
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