File: Hardware/Basic/Top/BuddyBand-BASIC-TOP.sch (EAGLE design)
At the start: 51 parts, among them SW1 SWITCH.MOM, SW6 SWITCH.MOM, U2 NRF52832_MODULE_MDBT42, U4 PCF8523

Commit message: In process of working on Take 003 video.
Parts:
- removed SW6: SWITCH.MOM, LinnesLab-Switches:SWITCH.MOM
- added C22: 100n, LinnesLab-Passives:CAPACITOR0603
- added C23, C24: 47p, LinnesLab-Passives:CAPACITOR0603
- added J1: (no value), LinnesLab-Connectors:CONN_07-1.27MM
- added JP2: (no value), LinnesLab-Switches:JUMPER-SMT_2_NO_SILK
- added LED5: RED, LinnesLab-LED:LED0603
- added LED6: YELLOW, LinnesLab-LED:LED0603
- added R1, R2: 0, LinnesLab-Passives:RESISTOR0603
- added R17, R18: 27, LinnesLab-Passives:RESISTOR0603
- added R19, R20: 1k, LinnesLab-Passives:RESISTOR0603
- added SW2: SWITCH.MOM, LinnesLab-Switches:SWITCH.MOM
- added U5: FT231XS, LinnesLab-DigitalIC:FT231XS
- R8, R9: value 10k -> 10K
- renumbered LDO2 to LDO1
Connections:
- net DC.OLED renamed D4/DC.OLED
- removed net BATT: R13.1, R14.2
- removed net CD1: SD2.CARD_DETECT
- removed net CHRG.STAT: CHRG2.STAT, R12.1
- removed net CS.OLED: U3./CS
- removed net RESET.OLED: U3./RES
- removed net RXD: U2.P0.08
- removed net SD.CS: SD2.CS
- removed net SW1: SW1.1, SW6.1
- removed net TXD: U2.P0.06
- new net !CTS: JP2.2, U5.!CTS
- new net A4/BATT: R13.1, R14.2, U2.P0.28/AIN4
- new net A6/TIA: J1.6, U2.P0.30/AIN6
- new net A7/PPG: J1.7, U2.P0.31/AIN7
- new net D11/SW1: SW1.1, U2.P0.11
- new net D15/SW2: SW2.1, U2.P0.15
- new net D16/CS.OLED: U2.P0.16, U3./CS
- new net D27/CHRG.STATUS: CHRG2.STAT, R12.1, U2.P0.27
- new net D29/LED.CTRL: J1.5, U2.P0.29/AIN5
- new net D3/RESET.OLED: U2.P0.03/AIN1, U3./RES
- new net D5/CD1: SD2.CARD_DETECT, U2.P0.05/AIN3
- new net D7/SD.CS: SD2.CS, U2.P0.07
- new net FT3V3: U5.3V3OUT
- new net N$16: U2.P0.04/AIN2
- new net N$23: R17.2, U5.USBDM
- new net N$24: R18.2, U5.USBDP
- new net N$25: LED5.C, R19.2
- new net N$26: LED6.C, R20.2
- new net RXD.FT: R2.1, U5.RXD
- new net RXD.NFR: R1.2, U2.P0.08
- new net RXLED: R19.1, U5.CBUS1
- new net TXD.FT: R1.1, U5.TXD
- new net TXD.NFR: R2.2, U2.P0.06
- new net TXLED: R20.1, U5.CBUS2
- net 3.3V: now also C22.2, J1.4, LED5.A, LED6.A, U5.!RESET, U5.VCCIO
- net DTR: now also U5.!DTR
- net GND: now also C22.1, C23.2, C24.1, J1.3, JP2.1, SW2.3, SW2.4, U5.GND@16, U5.GND@6; no longer SW6.3, SW6.4
- net SCL: now also J1.2, R9.1; no longer R8.1
- net SDA: now also J1.1, R8.1; no longer R9.1
- net USB+: now also C23.1, R18.1
- net USB-: now also C24.2, R17.1
- net V_USB: now also U5.VCC
Other:
- note added: "Analog Inputs Battery monitor Analog Inputs Analog Outputs"
- note added: "Connect to bottom board"
- note added: "Digital Output"
- note added: "Digital Outputs CS.OLED RESET.OLED DC.OLED Digital Inputs 3 x buttons Charge Status"
- note added: "FTDI Serial-to-USB Converter"
- note added: "I don't remember if CTS needs to be grounded or left floating so here's a jumper to ground so it can be configued either way dynamically."
- note added: "Notes:"
- note added: "TXD goes to RX on the other device RXD goes to TX on the other device"
- note removed: "Digital Outputs CS.OLED RESET.OLED DC.OLED Digital Inputs 3 x buttons Charge Status Analog Inputs Battery monitor Analog Inputs Analog Outputs"
- moved on the sheet: R8, R9, SW1, U4, XTAL3

Commit message: Finished take 5 working on take 6
Parts:
- removed C10, C11: 300p, LinnesLab-Passives:CAPACITOR0603
- removed C21: 4.7u, LinnesLab-Passives:CAPACITOR0603
- removed C23: 47p, LinnesLab-Passives:CAPACITOR0603
- removed D4: (no value), LinnesLab-DiscreteSemi:SCHOTTKY-USC
- removed R19, R20: 1k, LinnesLab-Passives:RESISTOR0603
- removed R9: 10K, LinnesLab-Passives:RESISTOR0603
- removed U3: (no value), LinnesLab-Displays:DISP_OLED_UG-2864HSWEG01-NO-WRAPAROUND
- removed XTAL3: 32.7680kHz, LinnesLab-Clocks:CRYSTALECS-.327-12.5-12-C-TR
- added C3: 1u, LinnesLab-Passives:CAPACITOR0603
- added D3: (no value), LinnesLab-DiscreteSemi:SCHOTTKY-USC
- added R10: 1k, LinnesLab-Passives:RESISTOR0603
- added R16: 10k, LinnesLab-Passives:RESISTOR0603
- C12: value 10u -> 1u; device LinnesLab-Passives:CAPACITOR0805 -> LinnesLab-Passives:CAPACITOR0603
- C13: value 2.2uF -> 4.7u; device LinnesLab-Passives:CAPACITOR0402 -> LinnesLab-Passives:CAPACITOR0603
- C15: value 2.2uF -> 10uF; device LinnesLab-Passives:CAPACITOR0402 -> LinnesLab-Passives:CAPACITOR0603
- C16: value 10uF -> 2.2uF; device LinnesLab-Passives:CAPACITOR0603 -> LinnesLab-Passives:CAPACITOR0402
- C2: value 1u -> 47p
- C20: value 4.7u -> 2.2uF; device LinnesLab-Passives:CAPACITOR0603 -> LinnesLab-Passives:CAPACITOR0402
- C5: value 1u -> 10u; device LinnesLab-Passives:CAPACITOR0603 -> LinnesLab-Passives:CAPACITOR0805
- C6: value 1u -> (none)
- C7: value 1u -> 4.7u
- C8: value (none) -> 1u
- R1, R2: value 0 -> 10K
- R11: value (none) -> 100k
- R13, R14: value 100k -> 0
- R15: value 100k -> 1k
- R17: value 27 -> 10k
- R18: value 27 -> 390k
- R3, R4: value 1k -> 27
- R5: value 10k -> 100k
- R6: value 10k -> 1k
- R7: value 390k -> 1k
- R8: value 10K -> (none)
- SW1, SW2: value SWITCH.MOM -> (none); device LinnesLab-Switches:SWITCH.MOM -> LinnesLab-Switches:SPST-PTS830GG140-COPY.1-3
- SW3, SW4: value (none) -> SWITCH.MOM; device LinnesLab-Switches:SPST-PTS830GG140-COPY.1-3 -> LinnesLab-Switches:SWITCH.MOM
- U4: value PCF8523 -> (none); device LinnesLab-Clocks:PCF8523 -> LinnesLab-Displays:DISP_OLED_UG-2864HSWEG01-NO-WRAPAROUND; DIGIKEY 568-5306-1-ND -> (none); I2C_ADDRESS 0x68h -> (none); MFN PCF8523T/1,118 -> (none); MFN_MANUFACTURER NXP USA Inc. -> (none)
- renumbered C22 to C4, C24 to C1, CHRG2 to CHRG1, CORTEX1 to DEBUG1, D5 to D2, JP2 to JP1, L2 to L1, LED5 to LED1, LED6 to LED2, SD2 to SD1, U5 to U1, USB2 to USB1, XTAL2 to XTAL1
Connections:
- removed net N$19: U4.OSCO, XTAL3.1
- removed net N$20: U4.OSCI, XTAL3.2
- net 3.3V: now also C12.1, C20.2, C5.2, D3.C, R1.2, R16.2, R2.2, U4.VBAT; no longer C12.2, C17.2, C2.1, C6.1, D1.C, R15.2, R5.2, R8.2, R9.2, U3.VBAT, U3.VDD
- net A4/BATT: now also R11.1, R12.2; no longer R13.1, R14.2
- net D11/SW1: now also SW3.1; no longer SW1.1
- net D15/SW2: now also SW4.1; no longer SW2.1
- net D16/CS.OLED: now also U4./CS; no longer U3./CS
- net D27/CHRG.STATUS: now also R5.1; no longer R12.1
- net D3/RESET.OLED: now also U4./RES; no longer U3./RES
- net D4/DC.OLED: now also U4.DC/I2C_SA0; no longer U3.DC/I2C_SA0
- net DFU: now also SW1.B; no longer SW3.B
- net GND: now also C12.2, C13.2, C15.1, C20.1, C3.2, C6.1, C7.1, R12.1, R17.1, R18.2, R8.1, SW1.A, SW2.B, SW3.3, SW4.3, U4.BS0, U4.BS2, U4.NC(GND)@1, U4.NC(GND)@2, U4.VLSS; no longer C10.2, C11.2, C12.1, C16.1, C18.1, C20.2, C21.1, C23.2, C6.2, C7.2, R11.1, R14.1, R15.1, R6.1, R7.2, SW1.3, SW1.4, SW2.3, SW2.4, SW3.A, SW4.B, U3.BS0, U3.BS2, U3.NC(GND)@1, U3.NC(GND)@2, U3.VLSS, U3.VSS
- net LED1: now also R10.2; no longer R3.2
- net LED2: now also R15.2; no longer R4.2
- net MOSI: now also U4.D1/SPI_SDIN/I2C_SDA; no longer U3.D1/SPI_SDIN/I2C_SDA
- net N$1: now also R17.2, U4.BS1; no longer R6.2, U3.BS1
- net N$10: now also R15.1; no longer R4.1
- net N$12: now also C3.1; no longer C7.1
- net N$13: now also C15.2, U4.VCC; no longer C16.2, U3.VCC
- net N$15: now also C17.2, U4.VCOMH; no longer C18.2, U3.VCOMH
- net N$17: now also R8.2; no longer R11.2
- net N$2: now also R18.1, U4.IREF; no longer R7.1, U3.IREF
- net N$23: now also R3.2; no longer R17.2
- net N$24: now also R4.2; no longer R18.2
- net N$25: now also R6.2; no longer R19.2
- net N$26: now also R7.2; no longer R20.2
- net N$3: now also C18.2, U4.C2P; no longer C13.2, U3.C2P
- net N$4: now also C6.2; no longer C8.2
- net N$5: now also C18.1, U4.C2N; no longer C13.1, U3.C2N
- net N$7: now also C16.2, U4.C1P; no longer C15.2, U3.C1P
- net N$8: now also C16.1, U4.C1N; no longer C15.1, U3.C1N
- net N$9: now also R10.1; no longer R3.1
- net P0.09/NFC1: no longer C11.1
- net P0.10/NFC2: no longer C10.1
- net RESET: now also D3.A, R16.1, SW2.A; no longer D1.A, R5.1, SW4.A
- net RXD.FT: now also R14.1; no longer R2.1
- net RXD.NFR: now also R13.2; no longer R1.2
- net RXLED: now also R6.1; no longer R19.1
- net SCK: now also U4.D0/SPI_SCLK/I2C_SCK; no longer U3.D0/SPI_SCLK/I2C_SCK
- net SCL: now also R2.1; no longer R9.1, U4.SCL
- net SDA: now also R1.1; no longer R8.1, U4.SDA
- net TXD.FT: now also R13.1; no longer R1.1
- net TXD.NFR: now also R14.2; no longer R2.2
- net TXLED: now also R7.1; no longer R20.1
- net USB+: now also C2.1, R4.1; no longer C23.1, R18.1
- net USB-: now also R3.1; no longer R17.1
- net VIN: now also C7.2, C8.2, D1.C, R5.2; no longer C21.2, C5.2, D4.C, R12.2
- net VLIPO: now also C13.1, D1.A, R11.2; no longer C20.1, D4.A, R13.2
Other:
- note removed: "Back-up battery if desired"
- note removed: "I2C Address = 0x68h"
- note removed: "Real-Time Clock"
- moved on the sheet: C12, C13, C15, C16, C17, C18, C2, C20, C5, C6, C7, C8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

Commit message: doing take 7. have trouble with wiring
Parts:
- removed SD1: (no value), LinnesLab-Connectors:MICROSD
Connections:
- removed net A6/TIA: J1.6, U2.P0.30/AIN6
- removed net A7/PPG: J1.7, U2.P0.31/AIN7
- removed net CD2: SD1.CARD_DETECT1
- removed net D29/LED.CTRL: J1.5, U2.P0.29/AIN5
- removed net N$16: U2.P0.04/AIN2
- new net A5/TIA: J1.6, U2.P0.29/AIN5
- new net A7/BATT: R11.1, R12.2, U2.P0.31/AIN7
- new net D30/LED.CTRL: J1.5, U2.P0.30/AIN6
- net 3.3V: no longer SD1.VDD
- net A4/BATT: now also J1.7; no longer R11.1, R12.2
- net D4/DC.OLED: now also U2.P0.04/AIN2
- net D5/CD1: no longer SD1.CARD_DETECT
- net D7/SD.CS: no longer SD1.CS
- net GND: no longer SD1.GND, SD1.GND1, SD1.VSS
- net MISO: no longer SD1.DATA_OUT
- net MOSI: no longer SD1.DATA_IN
- net SCK: no longer SD1.SCLK
Other:
- note removed: "Connect MISO, MOSI, and SCK to appropriate pins on microcontroller. Those are SPI pins and are generally prespecified. You have more flexibility with the SD.CS pin."
- note removed: "SD Card"
